File: kicad/hackaclock/hackaclock.kicad_sch (KiCad schematic)
At the start: 0 parts

Commit message: Added schematic
Parts:
- added BZ1: Buzzer, Buzzer_Beeper:Buzzer_12x9.5RM7.6, symbol Device:Buzzer
- added H1, H3, H4, H5: MountingHole, MountingHole:MountingHole_3.2mm_M3, symbol Mechanical:MountingHole
- added J1: Conn_01x08_Pin, Connector_PinSocket_2.54mm:PinSocket_1x08_P2.54mm_Vertical, symbol Connector:Conn_01x08_Pin
- added SW1, SW2, SW3, SW4, SW5, SW6: SW_Push, Button_Switch_Keyboard:SW_Cherry_MX_1.00u_PCB, symbol Switch:SW_Push
- added U1: XIAO-ESP32-C3-SMD, Seeed_Studio_XIAO_Series:XIAO-ESP32-C3-DIP, symbol Seeed_Studio_XIAO_Series.kicad_sym:XIAO-ESP32-C3-SMD
Connections:
- new net: SW2.2, U1.2 (D1)
- new net: SW4.2, U1.4 (D3)
- new net: BZ1.1 (+), U1.8 (D7)
- new net: SW5.2, U1.5 (D4)
- new net: SW6.2, U1.6 (D5)
- new net: SW3.2, U1.3 (D2)
- new net: SW1.2, U1.1 (D0)
- new net +3V3: J1.2 (Pin_2), J1.5 (Pin_5), U1.12 (3V3_OUT)
- new net CS: J1.7 (Pin_7), U1.7 (D6)
- new net DC: J1.6 (Pin_6), U1.9 (D8)
- new net GND: BZ1.2 (-), J1.1 (Pin_1), J1.8 (Pin_8), SW1.1, SW2.1, SW3.1, SW4.1, SW5.1, SW6.1, U1.13 (GND), U1.18 (GND), U1.22 (GND)
- new net SCL: J1.3 (Pin_3), U1.10 (D9/BOOT)
- new net SDA: J1.4 (Pin_4), U1.11 (D10)
- no-connect marks 0 -> 7
